File: hardware/TommyPROM-8755A Nano.sch (EAGLE design)
At the start: 14 parts, among them Q1 2N3904, Q2 2N3906

Commit message: Fix schematic label errors and pin assignments on 8755A device to match the schematic
Connections:
- removed net CE1/PROG: IC1.CE2, R1.2, U$2.A2
- new net CE1/PRG: IC1.PRG/!CE1, R3.2, U$2.A0
- net CE2: now also IC1.CE2, R1.2, U$2.A2; no longer IC1.PRG/!CE1, R3.2, U$2.A0
Changed lines of the file:
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@@
 </segment>
 </net>
-<net name="CE2" class="0">
+<net name="CE1/PRG" class="0">
 <segment>
 <wire x1="15.24" y1="114.3" x2="-30.48" y2="114.3" width="0.1524" layer="91"/>
@@
 </segment>
 </net>
-<net name="CE1/PROG" class="0">
+<net name="CE2" class="0">
 <segment>
 <wire x1="15.24" y1="109.22" x2="-25.4" y2="109.22" width="0.1524" layer="91"/>
