File: schematics/TommyPROM32/TommyPROM32.kicad_pcb (KiCad board)
At the start: 2 copper layers, 100 x 100 mm, 27 parts, among them J1 left, J10 GND, J11 VPP out, J12 D13, J13 VCC, J14 GND, J2 right, J3 PWR28, J4 PWR24, J5 high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

Commit message: V2.0 of the TommyPROM32 board
Parts:
- added C4: 0.1uF, Capacitor_THT:C_Disc_D3.0mm_W1.6mm_P2.50mm, F.Cu at (122.3, 104.8)
- added C5: 0.1uF, Capacitor_THT:C_Disc_D3.0mm_W1.6mm_P2.50mm, F.Cu at (139.2, 104.8)
- added D3: 1N5818, Diode_THT:D_DO-41_SOD81_P10.16mm_Horizontal, F.Cu at (147.3, 112.8)
- added D4: 1N5818, Diode_THT:D_DO-41_SOD81_P10.16mm_Horizontal, F.Cu at (141.3, 112.9)
- added J15: Tie, Connector_PinHeader_2.54mm:PinHeader_1x04_P2.54mm_Vertical, F.Cu at (62.4, 48.7)
- added J16: Tie, Connector_PinHeader_2.54mm:PinHeader_1x04_P2.54mm_Vertical, F.Cu at (140.2, 48.7)
- added J17: high, Connector_PinHeader_2.54mm:PinHeader_1x01_P2.54mm_Vertical, F.Cu at (141.3, 129.9)
- added J18: VPP out 2, Connector_PinHeader_2.54mm:PinHeader_1x02_P2.54mm_Vertical, F.Cu at (144.3, 104.8)
- added J19: GND, Connector_PinHeader_2.54mm:PinHeader_1x01_P2.54mm_Vertical, F.Cu at (134.1, 129.9)
- added SW2: SW_SPDT, digikey-footprints:Switch_Slide_11.6x4mm_EG1218, F.Cu at (135.1, 115.5)
- J11: value VPP out -> VPP out 1; footprint Connector_PinHeader_2.54mm:PinHeader_1x01_P2.54mm_Vertical -> Connector_PinHeader_2.54mm:PinHeader_1x02_P2.54mm_Vertical
- J13: value VCC -> low; footprint Connector_PinHeader_2.54mm:PinHeader_1x01_P2.54mm_Vertical -> Connector_PinHeader_2.54mm:PinHeader_1x02_P2.54mm_Vertical
- J6: footprint Connector_PinHeader_2.54mm:PinHeader_1x01_P2.54mm_Vertical -> Connector_PinHeader_2.54mm:PinHeader_1x02_P2.54mm_Vertical
- J7, J8: value VCC -> +5V
- moved R1 21.9 mm to (72.7, 100.0), turned to 180 degrees
- moved J14 21.4 mm to (127.6, 129.9)
- moved SW1 19.5 mm to (126.5, 115.5)
- moved R2 17.7 mm to (72.7, 103.0), turned to 180 degrees
- moved J12 16.8 mm to (58.6, 96.8)
- moved J11 15.1 mm to (117.2, 104.8)
- moved J6 14.8 mm to (114.2, 129.9), turned to 270 degrees
- moved D1 14.8 mm to (114.2, 112.9)
- moved D2 14.8 mm to (120.2, 112.9)
- moved J5 14.7 mm to (120.2, 129.9)
- moved R3 13.5 mm to (72.7, 106.0), turned to 180 degrees
- moved A1 13.1 mm to (100.9, 112.9)
- moved J10 11.6 mm to (140.2, 57.8), turned to 90 degrees
- moved J8 11.2 mm to (140.2, 39.6), turned to 90 degrees
- moved J9 6.57 mm to (62.4, 57.9), turned to 90 degrees
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- renumbered D2 to D1, D3 to D2
Connections:
- A1 pad 27: VCC -> +5V
- C1 pad 1: VCC -> +5V
- C2 pad 1: VCC -> +5V
- C3 pad 1: VCC -> +5V
- D1 pad 1: Net-(D2-Pad1) -> Net-(C4-Pad1)
- D2 pad 1: Net-(D2-Pad1) -> Net-(C4-Pad1)
- J11 pad 1: Net-(D2-Pad1) -> Net-(C4-Pad1)
- J13 pad 1: VCC -> Net-(D3-Pad2)
- J2 pad 2: VCC -> +5V
- J3 pad 1: VCC -> +5V
- J4 pad 1: VCC -> +5V
- J7 pad 1: VCC -> +5V
- J7 pad 2: VCC -> +5V
- J7 pad 3: VCC -> +5V
- J7 pad 4: VCC -> +5V
- J8 pad 1: VCC -> +5V
- J8 pad 2: VCC -> +5V
- J8 pad 3: VCC -> +5V
- J8 pad 4: VCC -> +5V
- R1 pad 1: VCC -> +5V
- R2 pad 1: VCC -> +5V
- R3 pad 1: VCC -> +5V
- U1 pad 14: VCC -> +5V
- U1 pad 2: VCC -> +5V
- U1 pad 9: VCC -> +5V
- U2 pad 14: VCC -> +5V
- U2 pad 2: VCC -> +5V
- U2 pad 9: VCC -> +5V
Routing:
- net ~OE: track 118.8 -> 140.1 mm, vias 1 -> 2
- net Net-(C4-Pad1): track 0.00 -> 21.2 mm
- net Net-(C5-Pad1): track 0.00 -> 21.1 mm
- net ~CE: track 110.4 -> 130.1 mm, vias 1 -> 2
- net VCC: track 17.5 -> 0.00 mm
- net ~WE: track 126.9 -> 142.5 mm, vias 1 -> 2
- net /CLK-HI: track 71.0 -> 85.9 mm
- net Net-(D2-Pad1): track 14.5 -> 0.00 mm
- net Net-(J17-Pad1): track 0.00 -> 14.5 mm
- net Net-(A1-Pad16): track 21.4 -> 35.4 mm, vias 0 -> 1
- net +5V: track 0.00 -> 11.8 mm
- net A17: track 95.2 -> 106.5 mm, vias 1 -> 2
- net Net-(D4-Pad2): track 0.00 -> 10.1 mm
- net A18: track 66.1 -> 74.1 mm, vias 0 -> 1
- net /AD-BIT: track 128.5 -> 136.3 mm
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- added copper zone on B.Cu, net +5V
- removed copper zone on B.Cu, net VCC
Other:
- board text added: "+5V"
- board text added: "2022 v2.0"
- board text added: "VPP in 1"
- board text added: "VPP in 2"
- board text removed: "2022 v1.0"
- board text removed: "VPP in"
- board text removed: "VPP select"
