File: schematics/TommyPROM32/TommyPROM32.sch (KiCad schematic (older format))
At the start: 27 parts, among them J1 left, J10 GND, J11 VPP out, J12 D13, J13 VCC, J14 GND, J2 right, J3 PWR28, J4 PWR24, J5 VPP high in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

Commit message: V2.0 of the TommyPROM32 board
Parts:
- removed J13: VCC, Connector_PinHeader_2.54mm:PinHeader_1x01_P2.54mm_Vertical, symbol Connector_Generic:Conn_01x01
- added C4, C5: 0.1uF, Capacitor_THT:C_Disc_D3.0mm_W1.6mm_P2.50mm, symbol Device:C
- added D3, D4: 1N5818, Diode_THT:D_DO-41_SOD81_P10.16mm_Horizontal, symbol Diode:1N5818
- added J13: low, Connector_PinHeader_2.54mm:PinHeader_1x02_P2.54mm_Vertical, symbol Connector_Generic:Conn_01x02
- added J15, J16: Tie, Connector_PinHeader_2.54mm:PinHeader_1x04_P2.54mm_Vertical, symbol Connector_Generic:Conn_01x04
- added J17: high, Connector_PinHeader_2.54mm:PinHeader_1x01_P2.54mm_Vertical, symbol Connector_Generic:Conn_01x01
- added J18: VPP out 2, Connector_PinHeader_2.54mm:PinHeader_1x02_P2.54mm_Vertical, symbol Connector_Generic:Conn_01x02
- added J19: GND, Connector_PinHeader_2.54mm:PinHeader_1x01_P2.54mm_Vertical, symbol Connector_Generic:Conn_01x01
- added SW2: SW_SPDT, digikey-footprints:Switch_Slide_11.6x4mm_EG1218, symbol Switch:SW_SPDT
- J11: value VPP out -> VPP out 1; footprint Connector_PinHeader_2.54mm:PinHeader_1x01_P2.54mm_Vertical -> Connector_PinHeader_2.54mm:PinHeader_1x02_P2.54mm_Vertical; symbol Connector_Generic:Conn_01x01 -> Connector_Generic:Conn_01x02
- J5: value VPP high in -> high
- J6: value VPP low in -> low; footprint Connector_PinHeader_2.54mm:PinHeader_1x01_P2.54mm_Vertical -> Connector_PinHeader_2.54mm:PinHeader_1x02_P2.54mm_Vertical; symbol Connector_Generic:Conn_01x01 -> Connector_Generic:Conn_01x02
- J7, J8: value VCC -> +5V
- U3: value EEPROM -> SST39SF040
- renumbered D2 to D1, D3 to D2
Connections:
- net GND: now also C4.2, C5.2, J19.1 (Pin_1)
- net at D1.1 (K), D2.1 (K), J11.1 (Pin_1): now also J11.2 (Pin_2), C4.1
- net VCC renamed +5V
- net +5V: now also J6.2 (Pin_2), J13.2 (Pin_2)
- new net: J16.1 (Pin_1), J16.2 (Pin_2), J16.3 (Pin_3), J16.4 (Pin_4)
- new net: J15.1 (Pin_1), J15.2 (Pin_2), J15.3 (Pin_3), J15.4 (Pin_4)
- new net: J17.1 (Pin_1), SW2.2 (B)
- new net: D3.2 (A), J13.1 (Pin_1)
- new net: D4.2 (A), SW2.1 (A)
- new net: C5.1, D3.1 (K), D4.1 (K), J18.1 (Pin_1), J18.2 (Pin_2)
- no-connect marks 10 -> 11
Other:
- note added: "VPP In"
- moved on the sheet: A1, C1, C2, C3, D1, D2, J1, J12, J14, J2, J3, J4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
